File: PCB/io/io.kicad_pcb (KiCad board)
At the start: 2 copper layers, 100 x 70 mm, 98 parts, among them U1 PiPico, U10 PC847, U11 PC847, U12 PCA9635, U2 TPS7A2042, U3 ADG708BRUZ, U4 ADG708BRUZ, U5 MCP23017_SS, U6 74HCT245, U7 74HCT245, U8 MCP23017_SS, U9 PC847

Commit message: IO Board v1.0 rc0
Parts:
- removed LO1, LO10, LO11, LO12, LO2, LO3, LO4, LO5, LO6, LO7, LO8, LO9: Conn_01x02_Pin, Connector_JST:JST_XH_B2B-XH-A_1x02_P2.50mm_Vertical
- removed U12: PCA9635, Package_SO:TSSOP-28_4.4x9.7mm_P0.65mm
- removed U5: MCP23017_SS, Package_SO:SSOP-28_5.3x10.2mm_P0.65mm
- added CC3: 0.1uF, Capacitor_SMD:C_0603_1608Metric_Pad1.08x0.95mm_HandSolder, B.Cu at (130.8, 122.9)
- added CC4: 0.1uF, Capacitor_SMD:C_0603_1608Metric_Pad1.08x0.95mm_HandSolder, B.Cu at (117.8, 122.9)
- added CC5: 0.1uF, Capacitor_SMD:C_0603_1608Metric_Pad1.08x0.95mm_HandSolder, B.Cu at (121.4, 82.0)
- added CC6: 0.1uF, Capacitor_SMD:C_0603_1608Metric_Pad1.08x0.95mm_HandSolder, B.Cu at (142.1, 82.0)
- added CC7: 0.1uF, Capacitor_SMD:C_0603_1608Metric_Pad1.08x0.95mm_HandSolder, B.Cu at (141.9, 113.7)
- added J1: RGB Out, Connector_JST:JST_XH_B3B-XH-A_1x03_P2.50mm_Vertical, F.Cu at (182.0, 116.0)
- added J2: RGB End, Connector_JST:JST_XH_B3B-XH-A_1x03_P2.50mm_Vertical, F.Cu at (192.0, 116.0)
- added JP1: 5V, io:SolderJump, B.Cu at (110.8, 118.0)
- added JP2: 3.3V, io:SolderJump, B.Cu at (110.8, 116.2)
- added PWR1: 5V In, Connector_JST:JST_XH_B2B-XH-A_1x02_P2.50mm_Vertical, F.Cu at (161.0, 116.0)
- added PWR2: 5V In, Connector_JST:JST_XH_B2B-XH-A_1x02_P2.50mm_Vertical, F.Cu at (171.0, 116.0)
- added PWR3: 5V In, Connector_JST:JST_XH_B2B-XH-A_1x02_P2.50mm_Vertical, F.Cu at (161.0, 125.0)
- added PWR4: 5V In, Connector_JST:JST_XH_B2B-XH-A_1x02_P2.50mm_Vertical, F.Cu at (171.0, 125.0)
- added R13: 1K, Resistor_SMD:R_0603_1608Metric_Pad0.98x0.95mm_HandSolder, B.Cu at (107.5, 112.5)
- added R14: 1K, Resistor_SMD:R_0603_1608Metric_Pad0.98x0.95mm_HandSolder, B.Cu at (107.5, 111.0)
- added S1: ~, io:M3_Screw, F.Cu at (193.0, 76.0)
- added S2: ~, io:M3_Screw, F.Cu at (193.0, 134.0)
- added S3: ~, io:M3_Screw, F.Cu at (107.0, 87.0)
- added S4: ~, io:M3_Screw, F.Cu at (107.0, 123.0)
- RN1, RN2, RN3, RN4, RN5, RN6, RN7, RN8, RN9: footprint Resistor_SMD:R_Array_Concave_4x0603 -> io:R_Array_Convex_4x0805
- U1: value PiPico -> Pico_Trim; footprint io:RPi_Pico_SMD_Pins -> io:RPi_Pico_SMD_No_USB
- Z3: moved to B.Cu
- moved RN6 36.6 mm to (135.0, 128.0)
- moved RN8 28.0 mm to (169.5, 106.1), turned to 180 degrees
- moved Z2 18.3 mm to (130.0, 101.0)
- moved U11 17.0 mm to (193.5, 105.5)
- moved RN5 16.9 mm to (127.0, 128.0)
- moved RN7 15.3 mm to (153.5, 106.1), turned to 180 degrees
- moved Z1 14.0 mm to (130.0, 98.5)
- moved U10 13.0 mm to (177.5, 105.5)
- moved U6 5.70 mm to (123.0, 120.0)
- moved CC1 4.87 mm to (110.6, 96.0), turned to 0 degrees
- moved RN4 4.78 mm to (119.0, 128.0)
- moved CC2 4.54 mm to (110.6, 93.7)
- moved U4 4.51 mm to (144.0, 87.0), turned to 90 degrees
- moved U7 4.51 mm to (136.0, 120.0)
- moved U3 3.75 mm to (126.2, 87.0), turned to 90 degrees
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- renumbered LI1 to Li1, LI10 to Li10, LI11 to Li11, LI12 to Li12, LI2 to Li2, LI3 to Li3, LI4 to Li4, LI5 to Li5, LI6 to Li6, LI7 to Li7, LI8 to Li8, LI9 to Li9
Connections:
- RN1 pad 5: Net-(In4-Pin_2) -> Net-(In1-Pin_2)
- RN1 pad 6: Net-(In3-Pin_2) -> Net-(In2-Pin_2)
- RN1 pad 7: Net-(In2-Pin_2) -> Net-(In3-Pin_2)
- RN1 pad 8: Net-(In1-Pin_2) -> Net-(In4-Pin_2)
- RN2 pad 5: Net-(In8-Pin_2) -> Net-(In5-Pin_2)
- RN2 pad 6: Net-(In7-Pin_2) -> Net-(In6-Pin_2)
- RN2 pad 7: Net-(In6-Pin_2) -> Net-(In7-Pin_2)
- RN2 pad 8: Net-(In5-Pin_2) -> Net-(In8-Pin_2)
- RN3 pad 5: Net-(In12-Pin_2) -> Net-(In9-Pin_2)
- RN3 pad 6: Net-(In11-Pin_2) -> Net-(In10-Pin_2)
- RN3 pad 7: Net-(In10-Pin_2) -> Net-(In11-Pin_2)
- RN3 pad 8: Net-(In9-Pin_2) -> Net-(In12-Pin_2)
- RN7 pad 1: Net-(RN7-R1.1) -> /GA4
- RN7 pad 2: Net-(RN7-R2.1) -> /GA5
- RN7 pad 3: Net-(RN7-R3.1) -> /GA6
- RN7 pad 4: Net-(RN7-R4.1) -> /GA7
- RN8 pad 1: Net-(RN8-R1.1) -> /GA0
- RN8 pad 2: Net-(RN8-R2.1) -> /GA1
- RN8 pad 3: Net-(RN8-R3.1) -> /GA2
- RN8 pad 4: Net-(RN8-R4.1) -> /GA3
- RN9 pad 1: Net-(RN9-R1.1) -> /GB3
- RN9 pad 2: Net-(RN9-R2.1) -> /GB2
- RN9 pad 3: Net-(RN9-R3.1) -> /GB1
- RN9 pad 4: Net-(RN9-R4.1) -> /GB0
- U1 pad 1: unconnected-(U1-GPIO0-Pad1) -> /SDA
- U1 pad 10: unconnected-(U1-GPIO7-Pad10) -> /O5
- U1 pad 11: unconnected-(U1-GPIO8-Pad11) -> /O6
- U1 pad 12: unconnected-(U1-GPIO9-Pad12) -> /O7
- U1 pad 13: unconnected-(U1-GND-Pad13) -> GND
- U1 pad 14: unconnected-(U1-GPIO10-Pad14) -> /O8
- U1 pad 15: unconnected-(U1-GPIO11-Pad15) -> /O9
- U1 pad 16: unconnected-(U1-GPIO12-Pad16) -> /O10
- U1 pad 17: unconnected-(U1-GPIO13-Pad17) -> /O11
- U1 pad 18: unconnected-(U1-GND-Pad18) -> GND
- U1 pad 19: unconnected-(U1-GPIO14-Pad19) -> Net-(J1-Pin_2)
- U1 pad 2: unconnected-(U1-GPIO1-Pad2) -> /SCL
- U1 pad 3: unconnected-(U1-GND-Pad3) -> GND
- U1 pad 4: /SDA -> /O0
- U1 pad 5: /SCL -> /O1
- U1 pad 6: unconnected-(U1-GPIO4-Pad6) -> /O2
- U1 pad 7: unconnected-(U1-GPIO5-Pad7) -> /O3
- U1 pad 8: unconnected-(U1-GND-Pad8) -> GND
- U1 pad 9: unconnected-(U1-GPIO6-Pad9) -> /O4
- U10 pad 1: Net-(D5-K) -> Net-(D10-K)
- U10 pad 10: Net-(RN8-R4.1) -> /GA0
- U10 pad 12: Net-(RN8-R3.1) -> /GA1
- U10 pad 14: Net-(RN8-R2.1) -> /GA2
- U10 pad 16: Net-(RN8-R1.1) -> /GA3
- U10 pad 2: Net-(D5-A) -> Net-(D10-A)
- U10 pad 3: Net-(D6-K) -> Net-(D3-K)
- U10 pad 4: Net-(D6-A) -> Net-(D3-A)
- U10 pad 5: Net-(D7-K) -> Net-(D4-K)
- U10 pad 6: Net-(D7-A) -> Net-(D4-A)
- U10 pad 7: Net-(D8-K) -> Net-(D9-K)
- U10 pad 8: Net-(D8-A) -> Net-(D9-A)
- U11 pad 1: Net-(D9-K) -> Net-(D8-K)
- U11 pad 10: Net-(RN9-R4.1) -> /GB3
- U11 pad 12: Net-(RN9-R3.1) -> /GB2
- U11 pad 14: Net-(RN9-R2.1) -> /GB1
- U11 pad 16: Net-(RN9-R1.1) -> /GB0
- U11 pad 2: Net-(D9-A) -> Net-(D8-A)
- U11 pad 3: Net-(D10-K) -> Net-(D5-K)
- U11 pad 4: Net-(D10-A) -> Net-(D5-A)
- U11 pad 5: Net-(D11-K) -> Net-(D6-K)
- U11 pad 6: Net-(D11-A) -> Net-(D6-A)
- U11 pad 7: Net-(D12-K) -> Net-(D7-K)
- U11 pad 8: Net-(D12-A) -> Net-(D7-A)
- U6 pad 19: unconnected-(U6-CE-Pad19) -> GND
- U6 pad 2: Net-(U5-GPB0) -> /O0
- U6 pad 3: Net-(U5-GPB1) -> /O1
- U6 pad 4: Net-(U5-GPB2) -> /O2
- U6 pad 5: Net-(U5-GPB3) -> /O3
- U6 pad 6: Net-(U5-GPB4) -> /O4
- U6 pad 7: Net-(U5-GPB5) -> /O5
- U6 pad 8: Net-(U5-GPB6) -> /O6
- U6 pad 9: Net-(U5-GPB7) -> /O7
- U7 pad 19: unconnected-(U7-CE-Pad19) -> GND
- U7 pad 2: Net-(U5-GPA0) -> /O8
- U7 pad 3: Net-(U5-GPA1) -> /O9
- U7 pad 4: Net-(U5-GPA2) -> /O10
- U7 pad 5: Net-(U5-GPA3) -> /O11
- U7 pad 6: Net-(U5-GPA4) -> unconnected-(U7-A4-Pad6)
- U7 pad 7: Net-(U5-GPA5) -> unconnected-(U7-A5-Pad7)
- U7 pad 8: Net-(U5-GPA6) -> unconnected-(U7-A6-Pad8)
- U7 pad 9: Net-(U5-GPA7) -> unconnected-(U7-A7-Pad9)
- U8 pad 1: Net-(RN7-R1.1) -> /GB0
- U8 pad 18: unconnected-(U8-~{RESET}-Pad18) -> +3V3
- U8 pad 2: Net-(RN7-R2.1) -> /GB1
- U8 pad 21: Net-(RN9-R1.1) -> /GA0
- U8 pad 22: Net-(RN9-R2.1) -> /GA1
- U8 pad 23: Net-(RN9-R3.1) -> /GA2
- U8 pad 24: Net-(RN9-R4.1) -> /GA3
- U8 pad 25: unconnected-(U8-GPA4-Pad25) -> /GA4
- U8 pad 26: unconnected-(U8-GPA5-Pad26) -> /GA5
- U8 pad 27: unconnected-(U8-GPA6-Pad27) -> /GA6
- U8 pad 28: unconnected-(U8-GPA7-Pad28) -> /GA7
- U8 pad 3: Net-(RN7-R3.1) -> /GB2
- U8 pad 4: Net-(RN7-R4.1) -> /GB3
- U8 pad 5: Net-(RN8-R1.1) -> /GB4
- U8 pad 6: Net-(RN8-R2.1) -> /GB5
- U8 pad 7: Net-(RN8-R3.1) -> /GB6
- U8 pad 8: Net-(RN8-R4.1) -> /GB7
- U9 pad 1: Net-(D1-K) -> Net-(D12-K)
- U9 pad 10: Net-(RN7-R4.1) -> /GA4
- U9 pad 12: Net-(RN7-R3.1) -> /GA5
- U9 pad 14: Net-(RN7-R2.1) -> /GA6
- U9 pad 16: Net-(RN7-R1.1) -> /GA7
- U9 pad 2: Net-(D1-A) -> Net-(D12-A)
- U9 pad 3: Net-(D2-K) -> Net-(D1-K)
- U9 pad 4: Net-(D2-A) -> Net-(D1-A)
- U9 pad 5: Net-(D3-K) -> Net-(D2-K)
- U9 pad 6: Net-(D3-A) -> Net-(D2-A)
- U9 pad 7: Net-(D4-K) -> Net-(D11-K)
- U9 pad 8: Net-(D4-A) -> Net-(D11-A)
Routing:
- net VHAL: track 0.00 -> 162.2 mm, vias 0 -> 2
- net +3V3: track 0.00 -> 158.0 mm, vias 0 -> 4
- net VBUS: track 0.00 -> 140.3 mm, vias 0 -> 1
- net VRGB: track 0.00 -> 97.5 mm
- net /GB3: track 0.00 -> 70.1 mm
- net /GB2: track 0.00 -> 63.9 mm
- net /GA0: track 0.00 -> 58.3 mm
- net /GB1: track 0.00 -> 57.8 mm
- net GND: track 0.00 -> 57.1 mm, vias 0 -> 65
- net /GA1: track 0.00 -> 52.1 mm
- net /GB0: track 0.00 -> 48.5 mm
- net Net-(Out12-Pin_1): track 0.00 -> 47.2 mm
- net /SDA: track 0.00 -> 46.7 mm, vias 0 -> 2
- net /GA2: track 0.00 -> 46.0 mm
- net /SCL: track 0.00 -> 42.5 mm, vias 0 -> 2
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- added copper zone on B.Cu, net GND
- added copper zone on F.Cu, net GND
Other:
- board text added: "+ -"
- board text added: "+ ~ -"
- board text added: "- +"
- board text added: "Out Level"
- board text added: "~ -"
