File: PCB/io/io.kicad_sch (KiCad schematic)
At the start: 98 parts, among them U1 PiPico, U10 PC847, U11 PC847, U12 PCA9635, U2 TPS7A2042, U3 ADG708BRUZ, U4 ADG708BRUZ, U5 MCP23017_SS, U6 74HCT245, U7 74HCT245, U8 MCP23017_SS, U9 PC847

Commit message: IO Board v1.0 rc0
Parts:
- removed LI10, LI11, LI12, LI2, LI3, LI4, LI5, LI6, LI7, LI8, LI9, LO1, LO10, LO11, LO12, LO2, LO3, LO4, LO5, LO6, LO7, LO8, LO9: Conn_01x02_Pin, Connector_JST:JST_XH_B2B-XH-A_1x02_P2.50mm_Vertical, symbol Connector:Conn_01x02_Pin
- removed U1: PiPico, io:RPi_Pico_SMD_Pins, symbol io:PiPico
- removed U12: PCA9635, Package_SO:TSSOP-28_4.4x9.7mm_P0.65mm, symbol Driver_LED:PCA9635
- removed U5: MCP23017_SS, Package_SO:SSOP-28_5.3x10.2mm_P0.65mm, symbol Interface_Expansion:MCP23017_SS
- added CC3, CC4, CC5, CC6, CC7: 0.1uF, Capacitor_SMD:C_0603_1608Metric_Pad1.08x0.95mm_HandSolder, symbol Device:C
- added J1: RGB Out, Connector_JST:JST_XH_B3B-XH-A_1x03_P2.50mm_Vertical, symbol Connector:Conn_01x03_Pin
- added J2: RGB End, Connector_JST:JST_XH_B3B-XH-A_1x03_P2.50mm_Vertical, symbol Connector:Conn_01x03_Pin
- added JP1: 5V, io:SolderJump, symbol Jumper:Jumper_2_Open
- added JP2: 3.3V, io:SolderJump, symbol Jumper:Jumper_2_Open
- added Li10, Li11, Li12, Li2, Li3, Li4, Li5, Li6, Li7, Li8, Li9: Conn_01x02_Pin, Connector_JST:JST_XH_B2B-XH-A_1x02_P2.50mm_Vertical, symbol Connector:Conn_01x02_Pin
- added PWR1, PWR2, PWR3, PWR4: 5V In, Connector_JST:JST_XH_B2B-XH-A_1x02_P2.50mm_Vertical, symbol Connector:Conn_01x02_Pin
- added R13, R14: 1K, Resistor_SMD:R_0603_1608Metric_Pad0.98x0.95mm_HandSolder, symbol Device:R
- added S1, S2, S3, S4: ~, io:M3_Screw, symbol io:M3_Screw
- added U1: Pico_Trim, io:RPi_Pico_SMD_No_USB, symbol io:Pico_Trim
- RN1, RN2, RN3, RN4, RN5, RN6, RN7, RN8, RN9: footprint Resistor_SMD:R_Array_Concave_4x0603 -> io:R_Array_Convex_4x0805
- renumbered In4 to In1, In11 to In10, In10 to In11, In9 to In12, In3 to In2, In2 to In3, In1 to In4, In8 to In5, In7 to In6, In6 to In7, In5 to In8, In12 to In9, LI1 to Li1, U9 to U10, U11 to U10, U10 to U11, U11 to U9
Connections:
- net +3V3: now also U8.18 (~{RESET}), CC7.1, JP2.1 (A), R13.2, R14.2, U1.36 (3V3)
- net GND: now also U10.11, U10.13, U10.15, U10.9, U11.11, U11.13, U11.15, U11.9, U6.19 (CE), U7.19 (CE), U9.11, U9.13, U9.15, U9.9, CC3.2, CC4.2, CC5.2, CC6.2, CC7.2, J1.3 (Pin_3), J2.3 (Pin_3), PWR1.2 (Pin_2), PWR2.2 (Pin_2), PWR3.2 (Pin_2), PWR4.2 (Pin_2), U1.13 (GND), U1.18 (GND), U1.23 (GND), U1.28 (GND), U1.3 (GND), U1.33 (AGND), U1.38 (GND), U1.8 (GND); no longer U10.11, U10.13, U10.15, U10.9, U11.11, U11.13, U11.15, U11.9, U9.11, U9.13, U9.15, U9.9
- net MUX_0: now also U1.26 (GPIO20)
- net MUX_1: now also U1.27 (GPIO21)
- net MUX_2: now also U1.29 (GPIO22)
- net SCL: now also R13.1, U1.2 (GPIO1)
- net SDA: now also R14.1, U1.1 (GPIO0)
- net VBUS: now also JP1.1 (A), PWR1.1 (Pin_1), PWR2.1 (Pin_1), PWR3.1 (Pin_1), PWR4.1 (Pin_1), U1.40 (VBUS)
- net VHAL: now also CC5.1, CC6.1
- net VO: now also CC3.1, CC4.1, JP1.2 (B), JP2.2 (B)
- net VRGB: now also J1.1 (Pin_1), J2.1 (Pin_1), U1.39 (VSYS)
- net at R8.1: now also Li8.1 (Pin_1)
- net at D8.2 (A): now also U11.2, Li8.2 (Pin_2); no longer U11.8
- net at D5.1 (K), R5.2: now also U11.3; no longer U11.1
- net at D5.2 (A): now also U11.4, Li5.2 (Pin_2); no longer U11.2
- net at D10.1 (K), R10.2: now also U10.1; no longer U10.3
- net at D10.2 (A): now also U10.2, Li10.2 (Pin_2); no longer U10.4
- net at D7.1 (K), R7.2: now also U11.7; no longer U11.5
- net at D7.2 (A): now also U11.8, Li7.2 (Pin_2); no longer U11.6
- net at D3.1 (K), R3.2: now also U10.3; no longer U10.5
- net at D3.2 (A): now also U10.4, Li3.2 (Pin_2); no longer U10.6
- net at D8.1 (K), R8.2: now also U11.1; no longer U11.7
- net at U4.8 (D), Z1.1 (K): now also U1.31 (GPIO26_ADC0)
- net at R4.1: now also Li4.1 (Pin_1)
- net at D4.1 (K), R4.2: now also U10.5; no longer U10.7
- net at R3.1: now also Li3.1 (Pin_1)
- net at U3.8 (D), Z2.1 (K): now also U1.32 (GPIO27_ADC1)
- net at D12.1 (K), R12.2: now also U9.1; no longer U9.7
- net at D12.2 (A): now also U9.2, Li12.2 (Pin_2); no longer U9.8
- net O0: now reaches U6.2 (A0)
- net O0: now also U1.4 (GPIO2)
- net O1: now reaches U6.3 (A1)
- net O1: now also U1.5 (GPIO3)
- net O8: now reaches U7.2 (A0)
- net O8: now also U1.14 (GPIO10)
- net O9: now reaches U7.3 (A1)
- net O9: now also U1.15 (GPIO11)
- net O10: now reaches U7.4 (A2)
- net O10: now also U1.16 (GPIO12)
- net O11: now reaches U7.5 (A3)
- net O11: now also U1.17 (GPIO13)
- net O2: now reaches U6.4 (A2)
- net O2: now also U1.6 (GPIO4)
- net O3: now reaches U6.5 (A3)
- net O3: now also U1.7 (GPIO5)
- net O4: now reaches U6.6 (A4)
- net O4: now also U1.9 (GPIO6)
- net O5: now reaches U6.7 (A5)
- net O5: now also U1.10 (GPIO7)
- net O6: now reaches U6.8 (A6)
- net O6: now also U1.11 (GPIO8)
- net O7: now reaches U6.9 (A7)
- net O7: now also U1.12 (GPIO9)
- net at R2.1: now also Li2.1 (Pin_1)
- net at D2.1 (K), R2.2: now also U9.5; no longer U9.3
- net at D4.2 (A): now also U10.6, Li4.2 (Pin_2); no longer U10.8
- net at D11.1 (K), R11.2: now also U9.7; no longer U9.5
- net at D11.2 (A): now also U9.8, Li11.2 (Pin_2); no longer U9.6
- net at D1.1 (K), R1.2: now also U9.3; no longer U9.1
- net at D1.2 (A), Li1.2 (Pin_2): now also U9.4; no longer U9.2
- net at Z3.1 (K): now also U1.35 (ADC_VREF)
- net at R10.1: now also Li10.1 (Pin_1)
- net GA4: now reaches U8.25 (GPA4)
- net GA4: now also RN7.1 (R1.1), U9.10
- net GA5: now reaches U8.26 (GPA5)
- net GA5: now also RN7.2 (R2.1), U9.12
- net GA6: now reaches U8.27 (GPA6)
- net GA6: now also RN7.3 (R3.1), U9.14
- net GA7: now reaches U8.28 (GPA7)
- net GA7: now also RN7.4 (R4.1), U9.16
- net at D2.2 (A): now also U9.6, Li2.2 (Pin_2); no longer U9.4
- net at R7.1: now also Li7.1 (Pin_1)
- net at R11.1: now also Li11.1 (Pin_1)
- net at D9.1 (K), R9.2: now also U10.7; no longer U10.1
- net at D9.2 (A): now also U10.8, Li9.2 (Pin_2); no longer U10.2
- net at R5.1: now also Li5.1 (Pin_1)
- net at R12.1: now also Li12.1 (Pin_1)
- net at R6.1: now also Li6.1 (Pin_1)
- net at D6.2 (A): now also U11.6, Li6.2 (Pin_2); no longer U11.4
- net at R9.1: now also Li9.1 (Pin_1)
- net at D6.1 (K), R6.2: now also U11.5; no longer U11.3
- new net: J1.2 (Pin_2), U1.19 (GPIO14)
- new net GA0: RN8.1 (R1.1), U10.10, U8.21 (GPA0)
- new net GA1: RN8.2 (R2.1), U10.12, U8.22 (GPA1)
- new net GA2: RN8.3 (R3.1), U10.14, U8.23 (GPA2)
- new net GA3: RN8.4 (R4.1), U10.16, U8.24 (GPA3)
- new net GB0: RN9.4 (R4.1), U11.16, U8.1 (GPB0)
- new net GB1: RN9.3 (R3.1), U11.14, U8.2 (GPB1)
- new net GB2: RN9.2 (R2.1), U11.12, U8.3 (GPB2)
- new net GB3: RN9.1 (R1.1), U11.10, U8.4 (GPB3)
- new net GB4: U8.5 (GPB4)
- new net GB5: U8.6 (GPB5)
- new net GB6: U8.7 (GPB6)
- new net GB7: U8.8 (GPB7)
- no-connect marks 0 -> 22
Other:
- moved on the sheet: CC1, CC2, D1, D10, D11, D12, D2, D3, D4, D5, D6, D7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
