File: PCB/button/button.kicad_sch (KiCad schematic)
At the start: 23 parts, among them J1 Conn_01x02_Socket, J2 Conn_01x03_Socket, J3 Lamp Seat, J4 In, J5 Out, J6 Lamp Seat, J7 Lamp Seat, SW1 SW_SPST, U1 SS49E_SOT23

Commit message: Button PCB v1.0 rc3
Parts:
- removed J1: Conn_01x02_Socket, Connector_PinHeader_2.54mm:PinHeader_1x02_P2.54mm_Vertical, symbol Connector:Conn_01x02_Socket
- added IR1: IR908-7C, button:IR908-7C, symbol button:IR908-7C
- added JP3: c, button:SolderJump, symbol Jumper:Jumper_2_Open
- added JP4: e, button:SolderJump, symbol Jumper:Jumper_2_Open
- added JP5: sw1, button:SolderJump, symbol Jumper:Jumper_2_Open
- added JP6: LEDP-V, button:SolderJump, symbol Jumper:Jumper_2_Open
- added JP7: sw2, button:SolderJump, symbol Jumper:Jumper_2_Open
- added PT1: PT908-7C, button:PT908-7C, symbol button:PT908-7C
- added R3: 200, Resistor_SMD:R_0805_2012Metric_Pad1.20x1.40mm_HandSolder, symbol Device:R
- added R4, R5: 200, Resistor_SMD:R_0805_2012Metric, symbol Device:R
- added SW2: (no value), button:SW_Kailh_Choc_V1V2, symbol Switch:SW_SPST
- added Z1: 3.3V, Diode_SMD:D_SOD-123F, symbol Device:D_Zener
- J2: footprint Connector_PinHeader_2.54mm:PinHeader_1x03_P2.54mm_Vertical -> button:SH1.0_3P_Solder_Combo
- J4: value In -> RGB In; footprint Connector_PinHeader_2.54mm:PinHeader_1x03_P2.54mm_Vertical -> button:SH1.0_3P_Solder_Combo
- J5: value Out -> RGB Out; footprint Connector_PinHeader_2.54mm:PinHeader_1x03_P2.54mm_Vertical -> button:SH1.0_3P_Solder_Combo
- SW1: value SW_SPST -> ~
Connections:
- net GND: now also IR1.1 (K), R5.1, SW2.2 (B), Z1.1 (K)
- net LED_P: now also JP6.1 (A)
- net Out: now also JP3.1 (A), JP4.1 (A), JP5.2 (B), JP7.2 (B), Z1.2 (A); no longer SW1.1 (A)
- net Vcc: now also JP6.2 (B), R3.2, R4.2
- new net: JP4.2 (B), PT1.1 (E), R5.2
- new net: IR1.2 (A), R3.1
- new net: JP7.1 (A), SW2.1 (A)
- new net: JP3.2 (B), PT1.2 (C), R4.1
- new net: JP5.1 (A), SW1.1 (A)
- no-connect marks 0 -> 1
Other:
- moved on the sheet: C1, C2, D3, D4, J2, J3, J4, J5, J6, SW1, U1

Commit message: Button and IO8 PCB
Parts:
- removed IR1: IR908-7C, button:IR908-7C, symbol button:IR908-7C
- removed PT1: PT908-7C, button:PT908-7C, symbol button:PT908-7C
- removed SW2: (no value), button:SW_Kailh_Choc_V1V2, symbol Switch:SW_SPST
- added SW2: Choc and IR Pair, button:SW_Kailh_Choc_IR_Combo, symbol button:SW_IR_COMBO
- J6, J7: value Lamp Seat -> Gold Finger
Connections:
- net GND: now also Z1.2 (A), SW2.2 (B), SW2.3 (K); no longer Z1.1 (K)
- net Out: now also Z1.1 (K); no longer Z1.2 (A)
- net at JP4.2 (B), R5.2: now also SW2.5 (E)
- net at R3.1: now also SW2.4 (A)
- net at JP7.1 (A): now also SW2.1 (A)
- net at JP3.2 (B), R4.1: now also SW2.6 (C)
Other:
- moved on the sheet: Z1
Changed lines of the file:
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@@
 			)
 		)
-		(property "Value" "Lamp Seat"
+		(property "Value" "Gold Finger"
 			(at 193.675 128.2699 0)
 			(effects
@@
 	)
 	(symbol
-		(lib_id "button:PT908-7C")
-		(at 113.665 85.725 0)
-		(unit 1)
-		(exclude_from_sim no)
-		(in_bom yes)
-		(on_board yes)
-		(dnp no)
-		(fields_autoplaced yes)
-		(property "Reference" "PT1"
-			(at 117.475 84.4549 0)
-			(effects
-				(font
-					(size 1.27 1.27)
-				)
-				(justify left)
-			)
-		)
-		(property "Value" "PT908-7C"
-			(at 117.475 86.9949 0)
-			(effects
-				(font
-					(size 1.27 1.27)
-				)
-				(justify left)
-			)
-		)
-		(property "Footprint" "button:PT908-7C"
-			(at 118.872 89.281 0)
-			(effects
-				(font
-					(size 1.27 1.27)
-				)
-				(justify left)
+		(lib_id "button:SW_IR_COMBO")
+		(at 163.83 49.53 0)
+		(unit 1)
+		(exclude_from_sim no)
+		(in_bom yes)
+		(on_board yes)
+		(dnp no)
+		(property "Reference" "SW2"
+			(at 163.83 46.355 0)
+			(effects
+				(font
+					(size 1.27 1.27)
+				)
+			)
+		)
+		(property "Value" "Choc and IR Pair"
+			(at 163.83 45.085 0)
+			(effects
+				(font
+					(size 1.27 1.27)
+				)
+				(hide yes)
+			)
+		)
+		(property "Footprint" "button:SW_Kailh_Choc_IR_Combo"
+			(at 163.576 51.054 0)
+			(effects
+				(font
+					(size 1.27 1.27)
+				)
 				(hide yes)
 			)
 		)
 		(property "Datasheet" ""
-			(at 113.665 85.725 0)
+			(at 163.83 49.53 0)
 			(effects
 				(font
@@
 		)
 		(property "Description" ""
-			(at 113.665 85.725 0)
+			(at 163.83 49.53 0)
 			(effects
 				(font
@@
 		(pin "1"
 		)
-		(instances
-			(project ""
-				(path "/6d76c26f-8ff0-4d96-92b3-afb2c3de8e4d"
-					(reference "PT1")
+		(pin "4"
+		)
+		(pin "6"
+		)
+		(pin "3"
+		)
+		(pin "5"
+		)
+		(instances
+			(project "button"
+				(path "/6d76c26f-8ff0-4d96-92b3-afb2c3de8e4d"
+					(reference "SW2")
 					(unit 1)
 				)
@@
 					(reference "#PWR03")
 					(unit 1)
+				)
+			)
+		)
+	)
+	(symbol
+		(lib_id "button:SW_IR_COMBO")
+		(at 90.805 91.44 90)
+		(unit 2)
+		(exclude_from_sim no)
+		(in_bom yes)
+		(on_board yes)
+		(dnp no)
+		(property "Reference" "SW2"
+			(at 95.25 91.44 90)
+			(effects
+				(font
+					(size 1.27 1.27)
+				)
+			)
+		)
+		(property "Value" "Choc and IR Pair"
+			(at 86.36 91.44 0)
+			(effects
+				(font
+					(size 1.27 1.27)
+				)
+				(hide yes)
+			)
+		)
+		(property "Footprint" "button:SW_Kailh_Choc_IR_Combo"
+			(at 92.329 91.694 0)
+			(effects
+				(font
+					(size 1.27 1.27)
+				)
+				(hide yes)
+			)
+		)
+		(property "Datasheet" ""
+			(at 90.805 91.44 0)
+			(effects
+				(font
+					(size 1.27 1.27)
+				)
+				(hide yes)
+			)
+		)
+		(property "Description" ""
+			(at 90.805 91.44 0)
+			(effects
+				(font
+					(size 1.27 1.27)
+				)
+				(hide yes)
+			)
+		)
+		(pin "2"
+		)
+		(pin "1"
+		)
+		(pin "4"
+		)
+		(pin "6"
+		)
+		(pin "3"
+		)
+		(pin "5"
+		)
+		(instances
+			(project "button"
+				(path "/6d76c26f-8ff0-4d96-92b3-afb2c3de8e4d"
+					(reference "SW2")
+					(unit 2)
 				)
 			)
@@
 	)
 	(symbol
+		(lib_id "button:SW_IR_COMBO")
+		(at 116.205 84.455 0)
+		(unit 3)
+		(exclude_from_sim no)
+		(in_bom yes)
+		(on_board yes)
+		(dnp no)
+		(property "Reference" "SW2"
+			(at 118.11 86.36 0)
+			(effects
+				(font
+					(size 1.27 1.27)
+				)
+			)
+		)
+		(property "Value" "Choc and IR Pair"
+			(at 116.205 80.01 0)
+			(effects
+				(font
+					(size 1.27 1.27)
+				)
+				(hide yes)
+			)
+		)
+		(property "Footprint" "button:SW_Kailh_Choc_IR_Combo"
+			(at 115.951 85.979 0)
+			(effects
+				(font
+					(size 1.27 1.27)
+				)
+				(hide yes)
+			)
+		)
+		(property "Datasheet" ""
+			(at 116.205 84.455 0)
+			(effects
+				(font
+					(size 1.27 1.27)
+				)
+				(hide yes)
+			)
+		)
+		(property "Description" ""
+			(at 116.205 84.455 0)
+			(effects
+				(font
+					(size 1.27 1.27)
+				)
+				(hide yes)
+			)
+		)
+		(pin "2"
+		)
+		(pin "1"
+		)
+		(pin "4"
+		)
+		(pin "6"
+		)
+		(pin "3"
+		)
+		(pin "5"
+		)
+		(instances
+			(project "button"
+				(path "/6d76c26f-8ff0-4d96-92b3-afb2c3de8e4d"
+					(reference "SW2")
+					(unit 3)
+				)
+			)
+		)
+	)
+	(symbol
 		(lib_id "power:VCC")
 		(at 99.695 31.75 0)
@@
 				(path "/6d76c26f-8ff0-4d96-92b3-afb2c3de8e4d"
 					(reference "#PWR011")
-					(unit 1)
-				)
-			)
-		)
-	)
-	(symbol
-		(lib_id "Switch:SW_SPST")
-		(at 163.83 49.53 0)
-		(unit 1)
-		(exclude_from_sim no)
-		(in_bom yes)
-		(on_board yes)
-		(dnp no)
-		(property "Reference" "SW2"
-			(at 163.83 46.355 0)
-			(effects
-				(font
-					(size 1.27 1.27)
-				)
-			)
-		)
-		(property "Value" ""
-			(at 163.83 45.72 0)
-			(effects
-				(font
-					(size 1.27 1.27)
-				)
-				(hide yes)
-			)
-		)
-		(property "Footprint" "button:SW_Kailh_Choc_V1V2"
-			(at 163.83 49.53 0)
-			(effects
-				(font
-					(size 1.27 1.27)
-				)
-				(hide yes)
-			)
-		)
-		(property "Datasheet" "~"
-			(at 163.83 49.53 0)
-			(effects
-				(font
-					(size 1.27 1.27)
-				)
-				(hide yes)
-			)
-		)
-		(property "Description" "Single Pole Single Throw (SPST) switch"
-			(at 163.83 49.53 0)
-			(effects
-				(font
-					(size 1.27 1.27)
-				)
-				(hide yes)
-			)
-		)
-		(pin "1"
-		)
-		(pin "2"
-		)
-		(instances
-			(project "button"
-				(path "/6d76c26f-8ff0-4d96-92b3-afb2c3de8e4d"
-					(reference "SW2")
 					(unit 1)
 				)
@@
 	)
 	(symbol
-		(lib_id "button:IR908-7C")
-		(at 90.805 90.17 90)
-		(unit 1)
-		(exclude_from_sim no)
-		(in_bom yes)
-		(on_board yes)
-		(dnp no)
-		(property "Reference" "IR1"
-			(at 95.25 90.17 90)
-			(effects
-				(font
-					(size 1.27 1.27)
-				)
-			)
-		)
-		(property "Value" "IR908-7C"
-			(at 98.425 92.075 90)
-			(effects
-				(font
-					(size 1.27 1.27)
-				)
-			)
-		)
-		(property "Footprint" "button:IR908-7C"
-			(at 86.36 90.17 0)
-			(effects
-				(font
-					(size 1.27 1.27)
-				)
-				(hide yes)
-			)
-		)
-		(property "Datasheet" ""
-			(at 90.805 91.44 0)
-			(effects
-				(font
-					(size 1.27 1.27)
-				)
-				(hide yes)
-			)
-		)
-		(property "Description" ""
-			(at 90.805 90.17 0)
-			(effects
-				(font
-					(size 1.27 1.27)
-				)
-				(hide yes)
-			)
-		)
-		(pin "1"
-		)
-		(pin "2"
-		)
-		(instances
-			(project ""
-				(path "/6d76c26f-8ff0-4d96-92b3-afb2c3de8e4d"
-					(reference "IR1")
-					(unit 1)
-				)
-			)
-		)
-	)
-	(symbol
 		(lib_id "power:GND")
 		(at 181.61 136.525 0)
@@
 	(symbol
 		(lib_id "Device:D_Zener")
-		(at 137.16 90.805 90)
+		(at 137.16 90.805 270)
 		(unit 1)
 		(exclude_from_sim no)
@@
 					(size 1.27 1.27)
 				)
-				(justify right)
+				(justify left)
 			)
 		)
@@
 					(size 1.27 1.27)
 				)
-				(justify right)
+				(justify left)
 			)
 		)
@@
 			)
 		)
-		(property "Value" "Lamp Seat"
+		(property "Value" "Gold Finger"
 			(at 58.42 139.6999 0)
 			(effects
